Commit message: Fixed inertial errors

File: mini_pupper_description/urdf/mini_pupper_description.urdf.xacro (robot description, xacro)
@@ -2,5 +2,5 @@
 <robot name="mini_pupper" xmlns:xacro="http://www.ros.org/wiki/xacro">
   <xacro:include filename="$(find mini_pupper_description)/urdf/materials.xacro" />
-  <!-- <xacro:include filename="$(find mini_pupper_description)/urdf/mini_pupper_description.trans" /> -->
+  <xacro:include filename="$(find mini_pupper_description)/urdf/mini_pupper_description.trans" />
   <link name="base_link">
     <visual>
@@ -20,7 +20,7 @@
   <link name="base_inertia">
     <inertial>
-      <origin xyz="-0.008866664732250966 0.0006462612742260995 -0.007154314406453802" rpy="0 0 0"/>
+      <origin xyz="-0.008867 0.000646 -0.007154" rpy="0 0 0"/>
       <mass value="0.09818420433466489"/>
-      <inertia ixx="5.2e-05" iyy="0.000244" izz="0.000252" ixy="1e-06" iyz="1e-06" ixz="-1e-05"/>
+      <inertia ixx="5.2003168e-05" iyy="2.437e-4" izz="2.523e-4" ixy="7.28047e-07" iyz="6.0331e-07" ixz="-9.716561e-06"/>
     </inertial>
   </link>
@@ -29,5 +29,5 @@
       <origin xyz="0.020109281613098752 0.002331771723067172 0.0064994497731911665" rpy="0 0 0"/>
       <mass value="0.020769030109708524"/>
-      <inertia ixx="2e-06" iyy="4e-06" izz="3e-06" ixy="0.0" iyz="0.0" ixz="0.0"/>
+      <inertia ixx="2.494e-06" iyy="3.736e-06" izz="3.223e-06" ixy="-7.659e-9" iyz="0.072e-9" ixz="-33.608e-9"/>
     </inertial>
     <visual>
@@ -49,5 +49,5 @@
       <origin xyz="-0.0031735030993243693 0.000986055889313886 -0.01798354657247523" rpy="0 0 0"/>
       <mass value="0.0019057729925096327"/>
-      <inertia ixx="0.0" iyy="0.0" izz="0.0" ixy="0.0" iyz="0.0" ixz="0.0"/>
+      <inertia ixx="0.462154e-6" iyy="0.481174e-6" izz="26.893e-9" ixy="3.117e-9" iyz="17.662e-9" ixz="-79.269e-9"/>
     </inertial>
     <visual>
@@ -69,5 +69,5 @@
       <origin xyz="0.006210627225594921 0.003455723027058405 -0.015013638057132746" rpy="0 0 0"/>
       <mass value="0.0011438144457690698"/>
-      <inertia ixx="1e-06" iyy="1e-06" izz="0.0" ixy="0.0" iyz="0.0" ixz="0.0"/>
+      <inertia ixx="0.484118e-6" iyy="0.567346e-06" izz="91.82e-9" ixy="-2.157e-9" iyz="4.945e-9" ixz="0.200546e-6"/>
     </inertial>
     <visual>
@@ -89,5 +89,5 @@
       <origin xyz="0.020106742599110078 -0.00233237781568562 0.006497900858401761" rpy="0 0 0"/>
       <mass value="0.020769549324466178"/>
-      <inertia ixx="2e-06" iyy="4e-06" izz="3e-06" ixy="0.0" iyz="0.0" ixz="0.0"/>
+      <inertia ixx="2.494e-06" iyy="3.736e-06" izz="3.223e-06" ixy="7.618e-9" iyz="0.098e-9" ixz="-37.629e-9"/>
     </inertial>
     <visual>
@@ -109,5 +109,5 @@
       <origin xyz="-0.00317137334512671 -0.000986627579459616 -0.01798392230653304" rpy="0 0 0"/>
       <mass value="0.0019057729924780605"/>
-      <inertia ixx="0.0" iyy="0.0" izz="0.0" ixy="0.0" iyz="0.0" ixz="0.0"/>
+      <inertia ixx="0.462172e-6" iyy="0.481174e-6" izz="26.874e-9" ixy="-3.114e-9" iyz="-17.663e-9" ixz="-79.218e-9"/>
     </inertial>
     <visual>
@@ -129,5 +129,5 @@
       <origin xyz="0.006211719758792998 -0.0034574884973188197 -0.01500899883342268" rpy="0 0 0"/>
       <mass value="0.001143490701517533"/>
-      <inertia ixx="1e-06" iyy="1e-06" izz="0.0" ixy="0.0" iyz="0.0" ixz="0.0"/>
+      <inertia ixx="0.484726e-6" iyy="0.567959e-06" izz="91.882e-9" ixy="2.056e-9" iyz="-4.954e-9" ixz="0.200706e-6"/>
     </inertial>
     <visual>
@@ -149,5 +149,5 @@
       <origin xyz="-0.020107177922528044 -0.0023288309787250286 0.006502376356642127" rpy="0 0 0"/>
       <mass value="0.020769549324363486"/>
-      <inertia ixx="2e-06" iyy="4e-06" izz="3e-06" ixy="0.0" iyz="0.0" ixz="0.0"/>
+      <inertia ixx="2.494e-06" iyy="3.736e-06" izz="3.223e-06" ixy="-7.639e-9" iyz="-0.378e-9" ixz="-37.624e-9"/>
     </inertial>
     <visual>
@@ -169,5 +169,5 @@
       <origin xyz="-0.0031709881638501275 -0.0009964344348111775 -0.017982726579309202" rpy="0 0 0"/>
       <mass value="0.0019057729926311429"/>
-      <inertia ixx="0.0" iyy="0.0" izz="0.0" ixy="0.0" iyz="0.0" ixz="0.0"/>
+      <inertia ixx="0.462172e-6" iyy="0.481155e-6" izz="26.893e-9" ixy="-3.158e-9" iyz="-17.911e-9" ixz="-79.911e-9"/>
     </inertial>
     <visual>
@@ -189,5 +189,5 @@
       <origin xyz="0.006208573190273861 -0.0034623583329196975 -0.015001217060300935" rpy="0 0 0"/>
       <mass value="0.0011440535724654094"/>
-      <inertia ixx="1e-06" iyy="1e-06" izz="0.0" ixy="0.0" iyz="0.0" ixz="0.0"/>
+      <inertia ixx="0.484539e-6" iyy="0.567687e-06" izz="91.857e-9" ixy="2.182e-9" iyz="-5.285e-9" ixz="0.200597e-6"/>
     </inertial>
     <visual>
@@ -209,5 +209,5 @@
       <origin xyz="-0.020109716415830967 0.0023317718989125207 0.006499556305653081" rpy="0 0 0"/>
       <mass value="0.020769030189864354"/>
-      <inertia ixx="2e-06" iyy="4e-06" izz="3e-06" ixy="0.0" iyz="0.0" ixz="0.0"/>
+      <inertia ixx="2.494e-06" iyy="3.736e-06" izz="3.223e-06" ixy="7.659e-9" iyz="-0.072e-9" ixz="-33.608e-9"/>
     </inertial>
     <visual>
@@ -229,5 +229,5 @@
       <origin xyz="-0.0031709879518865836 0.0009860564153100285 -0.01798392227051571" rpy="0 0 0"/>
       <mass value="0.0019057729925095609"/>
-      <inertia ixx="0.0" iyy="0.0" izz="0.0" ixy="0.0" iyz="0.0" ixz="0.0"/>
+      <inertia ixx="0.462172e-6" iyy="0.481174e-6" izz="26.874e-9" ixy="3.114e-9" iyz="17.663e-9" ixz="-79.218e-9"/>
     </inertial>
     <visual>
@@ -249,5 +249,5 @@
       <origin xyz="0.006208905683926957 0.0034523757482988054 -0.015005654191541921" rpy="0 0 0"/>
       <mass value="0.001144346207072784"/>
-      <inertia ixx="1e-06" iyy="1e-06" izz="0.0" ixy="0.0" iyz="0.0" ixz="0.0"/>
+      <inertia ixx="0.484492e-6" iyy="0.567176e-06" izz="91.41e-9" ixy="-2.023e-9" iyz="4.977e-9" ixz="0.200063e-6"/>
     </inertial>
     <visual>
@@ -309,5 +309,5 @@
       <origin xyz="-0.07276303117117414 -0.002323344081837563 -0.0010631239213060653" rpy="0 0 0"/>
       <mass value="0.004688613655947816"/>
-      <inertia ixx="0.0" iyy="1.5e-05" izz="1.6e-05" ixy="-1e-06" iyz="0.0" ixz="0.0"/>
+      <inertia ixx="0.203205e-6" iyy="1.5404404e-05" izz="1.5546403e-05" ixy="-0.625328e-06" iyz="42.901e-9" ixz="0.186346e-9"/>
     </inertial>
     <visual>
@@ -329,5 +329,5 @@
       <origin xyz="0.008233541174180986 -0.002138369786547657 -0.00030110978110910874" rpy="0 0 0"/>
       <mass value="0.0019746031301169403"/>
-      <inertia ixx="0.0" iyy="3e-06" izz="4e-06" ixy="0.0" iyz="0.0" ixz="0.0"/>
+      <inertia ixx="0.458176e-6" iyy="3.284711e-06" izz="3.720353e-06" ixy="-79.81e-9" iyz="4.793e-9" ixz="0.123862e-9"/>
     </inertial>
     <visual>
@@ -349,5 +349,5 @@
       <origin xyz="-0.004983173489839052 -2.855799938611403e-07 0.006488367917121082" rpy="0 0 0"/>
       <mass value="0.0014053107976262874"/>
-      <inertia ixx="0.0" iyy="0.0" izz="0.0" ixy="0.0" iyz="0.0" ixz="0.0"/>
+      <inertia ixx="41.992e-9" iyy="62.399e-9" izz="29.801e-9" ixy="0.0" iyz="0.0" ixz="1.625e-9"/>
     </inertial>
     <visual>
@@ -369,5 +369,5 @@
       <origin xyz="-0.004982788301465979 3.706995898918042e-06 0.006488719406103974" rpy="0 0 0"/>
       <mass value="0.0014053107976262874"/>
-      <inertia ixx="0.0" iyy="0.0" izz="0.0" ixy="0.0" iyz="0.0" ixz="0.0"/>
+      <inertia ixx="41.992e-9" iyy="62.399e-9" izz="29.801e-9" ixy="0.001e-9" iyz="-0.018e-9" ixz="1.625e-9"/>
     </inertial>
     <visual>
@@ -389,5 +389,5 @@
       <origin xyz="-0.004982788451759437 -2.855826620323798e-07 0.0064883680140642025" rpy="0 0 0"/>
       <mass value="0.0014053107976262874"/>
-      <inertia ixx="0.0" iyy="0.0" izz="0.0" ixy="0.0" iyz="0.0" ixz="0.0"/>
+      <inertia ixx="41.992e-9" iyy="62.399e-9" izz="29.801e-9" ixy="0.0" iyz="0.0" ixz="1.625e-9"/>
     </inertial>
     <visual>
@@ -409,5 +409,5 @@
       <origin xyz="-0.004983499344395154 -2.861132842799097e-07 0.006488888240325896" rpy="0 0 0"/>
       <mass value="0.0014053107976262874"/>
-      <inertia ixx="0.0" iyy="0.0" izz="0.0" ixy="0.0" iyz="0.0" ixz="0.0"/>
+      <inertia ixx="41.992e-9" iyy="62.399e-9" izz="29.801e-9" ixy="0.0" iyz="0.0" ixz="1.625e-9"/>
     </inertial>
     <visual>
@@ -429,5 +429,5 @@
       <origin xyz="0.002258882765982295 0.008667473212030541 -0.002747896746317195" rpy="0 0 0"/>
       <mass value="0.002573897544461238"/>
-      <inertia ixx="0.0" iyy="0.0" izz="0.0" ixy="0.0" iyz="0.0" ixz="0.0"/>
+      <inertia ixx="0.390582e-6" iyy="0.412423e-6" izz="0.246322e-6" ixy="24.632e-9" iyz="3.861e-9" ixz="54.103e-9"/>
     </inertial>
     <visual>
@@ -449,5 +449,5 @@
       <origin xyz="0.0022592683660053597 0.008667473212031727 -0.0027478967463174797" rpy="0 0 0"/>
       <mass value="0.002573897544461238"/>
-      <inertia ixx="0.0" iyy="0.0" izz="0.0" ixy="0.0" iyz="0.0" ixz="0.0"/>
+      <inertia ixx="0.390582e-6" iyy="0.412423e-6" izz="0.246322e-6" ixy="24.632e-9" iyz="3.861e-9" ixz="54.103e-9"/>
     </inertial>
     <visual>
@@ -469,5 +469,5 @@
       <origin xyz="0.002219644336096324 -0.008605630927951344 -0.002709000699399786" rpy="0 0 0"/>
       <mass value="0.002396251664132183"/>
-      <inertia ixx="0.0" iyy="0.0" izz="0.0" ixy="0.0" iyz="0.0" ixz="0.0"/>
+      <inertia ixx="0.364377e-6" iyy="0.38866e-6" izz="0.234177e-6" ixy="-23.674e-9" iyz="-3.338e-9" ixz="52.098e-9"/>
     </inertial>
     <visual>
@@ -489,5 +489,5 @@
       <origin xyz="0.0022200295152449145 -0.008607013686777375 -0.0027033986949916797" rpy="0 0 0"/>
       <mass value="0.002396251664132183"/>
-      <inertia ixx="0.0" iyy="0.0" izz="0.0" ixy="0.0" iyz="0.0" ixz="0.0"/>
+      <inertia ixx="0.364377e-6" iyy="0.388657e-6" izz="0.23418e-6" ixy="-23.645e-9" iyz="-3.422e-9" ixz="52.111e-9"/>
     </inertial>
     <visual>
@@ -509,5 +509,5 @@
       <origin xyz="-0.001747332142694763 0.00790352811362327 0.005364507913861985" rpy="0 0 0"/>
       <mass value="0.0022314211131891203"/>
-      <inertia ixx="1e-06" iyy="1e-06" izz="0.0" ixy="0.0" iyz="-0.0" ixz="-0.0"/>
+      <inertia ixx="0.862549e-06" iyy="0.991391e-06" izz="0.139046e-6" ixy="1.254e-9" iyz="-13.212e-9" ixz="-0.112903e-9"/>
     </inertial>
     <visual>
@@ -529,5 +529,5 @@
       <origin xyz="-0.001747730780760487 0.007903528639619323 0.005365117008527457" rpy="0 0 0"/>
       <mass value="0.0022314211131891203"/>
-      <inertia ixx="1e-06" iyy="1e-06" izz="0.0" ixy="0.0" iyz="-0.0" ixz="-0.0"/>
+      <inertia ixx="0.862549e-06" iyy="0.991391e-06" izz="0.139046e-6" ixy="1.254e-9" iyz="-13.212e-9" ixz="-0.112903e-9"/>
     </inertial>
     <visual>
@@ -549,5 +549,5 @@
       <origin xyz="-0.0018083907227202795 -0.007907075713007514 0.005388328467850496" rpy="0 0 0"/>
       <mass value="0.002201611562253873"/>
-      <inertia ixx="1e-06" iyy="1e-06" izz="0.0" ixy="-0.0" iyz="0.0" ixz="-0.0"/>
+      <inertia ixx="0.859857e-06" iyy="0.986828e-06" izz="0.137126e-6" ixy="-1.292e-9" iyz="13.109e-9" ixz="-0.111508e-9"/>
     </inertial>
     <visual>
@@ -569,5 +569,5 @@
       <origin xyz="-0.0018090055415128231 -0.007904339012704771 0.005392934920359041" rpy="0 0 0"/>
       <mass value="0.002201611562253873"/>
-      <inertia ixx="1e-06" iyy="1e-06" izz="0.0" ixy="-0.0" iyz="0.0" ixz="-0.0"/>
+      <inertia ixx="0.859857e-06" iyy="0.986842e-06" izz="0.137112e-6" ixy="-1.352e-9" iyz="12.645e-9" ixz="-0.111508e-9"/>
     </inertial>
     <visual>
