Commit message: Fixed proning in neutral pose

File: mini_pupper_description/urdf/mini_pupper_description.urdf (robot description, URDF)
Before this commit: robot mini_pupper, 32 links, 31 joints
Links:
- link Shell_Leg_Upper_LeftSide_1: mass 0.00223142111318912 -> 0.0022314211131891203
- link Shell_Leg_Upper_LeftSide_2: mass 0.00223142111318912 -> 0.0022314211131891203
- link Shell_Leg_Upper_RightSide_1: mass 0.0022016115622538724 -> 0.002201611562253873
- link Shell_Leg_Upper_RightSide_2: mass 0.0022016115622538724 -> 0.002201611562253873
Joints:
- joint lb1_lb2: axis 0.0 1.0 -0.0 -> 0.0 1.0 0.0
- joint lb2_lb3: axis 0.0 1.0 -0.0 -> 0.0 1.0 0.0; origin xyz=0.0 0.003 -0.05 rpy=0 0 0 -> xyz=-0.008682 0.003 -0.049241 rpy=0 0 0
- joint lb2_shell: origin xyz=0.0 0.003 -0.019 rpy=0 0 0 -> xyz=-0.003299 0.003 -0.018712 rpy=0 0 0
- joint lb3_foot: origin xyz=0.004524 0.00375 -0.059571 rpy=0 0 0 -> xyz=0.024625 0.00375 -0.05443 rpy=0 0 0
- joint lf1_lf2: axis 0.0 1.0 -0.0 -> 0.0 1.0 0.0
- joint lf2_lf3: axis 0.0 1.0 -0.0 -> 0.0 1.0 0.0; origin xyz=-6e-06 0.003 -0.05 rpy=0 0 0 -> xyz=-0.008689 0.003 -0.04924 rpy=0 0 0
- joint lf2_shell: origin xyz=-3e-06 0.003 -0.019 rpy=0 0 0 -> xyz=-0.003302 0.003 -0.018711 rpy=0 0 0
- joint lf3_foot: origin xyz=0.00453 0.00375 -0.05957 rpy=0 0 0 -> xyz=0.024632 0.00375 -0.054428 rpy=0 0 0
- joint rb2_rb3: origin xyz=0.0 -0.003028 -0.049998 rpy=0 0 0 -> xyz=-0.008682 -0.003027 -0.049239 rpy=0 0 0
- joint rb2_shell: origin xyz=0.0 -0.003011 -0.018998 rpy=0 0 0 -> xyz=-0.003299 -0.00301 -0.01871 rpy=0 0 0
- joint rb3_foot: origin xyz=0.004524 -0.003782 -0.059568 rpy=0 0 0 -> xyz=0.024625 -0.00378 -0.054428 rpy=0 0 0
- joint rf2_rf3: origin xyz=0.0 -0.003 -0.05 rpy=0 0 0 -> xyz=-0.008683 -0.003 -0.049241 rpy=0 0 0
- joint rf2_shell: origin xyz=0.0 -0.003 -0.019 rpy=0 0 0 -> xyz=-0.0033 -0.003 -0.018712 rpy=0 0 0
- joint rf3_foot: origin xyz=0.004524 -0.00375 -0.059571 rpy=0 0 0 -> xyz=0.024626 -0.00375 -0.05443 rpy=0 0 0

File: mini_pupper_description/urdf/mini_pupper_description.urdf.xacro (robot description, xacro)
@@ -29,5 +29,5 @@
       <origin xyz="0.020109281613098752 0.002331771723067172 0.0064994497731911665" rpy="0 0 0"/>
       <mass value="0.020769030109708524"/>
-      <inertia ixx="2e-06" iyy="4e-06" izz="3e-06" ixy="-0.0" iyz="-0.0" ixz="-0.0"/>
+      <inertia ixx="2e-06" iyy="4e-06" izz="3e-06" ixy="0.0" iyz="0.0" ixz="0.0"/>
     </inertial>
     <visual>
@@ -47,7 +47,7 @@
   <link name="lf2">
     <inertial>
-      <origin xyz="-2.5728896106275156e-06 0.0009860558893138652 -0.018261345499916863" rpy="0 0 0"/>
+      <origin xyz="-0.0031735030993243693 0.000986055889313886 -0.01798354657247523" rpy="0 0 0"/>
       <mass value="0.0019057729925096327"/>
-      <inertia ixx="0.0" iyy="0.0" izz="0.0" ixy="0.0" iyz="0.0" ixz="-0.0"/>
+      <inertia ixx="0.0" iyy="0.0" izz="0.0" ixy="0.0" iyz="0.0" ixz="0.0"/>
     </inertial>
     <visual>
@@ -67,10 +67,10 @@
   <link name="lf3">
     <inertial>
-      <origin xyz="0.0007046107744873437 0.0034550275861905885 -0.016225601428628958" rpy="0 0 0"/>
+      <origin xyz="0.006210627225594921 0.003455723027058405 -0.015013638057132746" rpy="0 0 0"/>
       <mass value="0.0011438144457690698"/>
-      <inertia ixx="1e-06" iyy="1e-06" izz="0.0" ixy="-0.0" iyz="0.0" ixz="0.0"/>
-    </inertial>
-    <visual>
-      <origin xyz="-0.052159 -0.044445 0.049943" rpy="0 0 0"/>
+      <inertia ixx="1e-06" iyy="1e-06" izz="0.0" ixy="0.0" iyz="0.0" ixz="0.0"/>
+    </inertial>
+    <visual>
+      <origin xyz="-0.043476 -0.044445 0.049183" rpy="0 0 0"/>
       <geometry>
         <mesh filename="package://mini_pupper_description/meshes/lf3.stl" scale="1 1 1"/>
@@ -79,5 +79,5 @@
     </visual>
     <collision>
-      <origin xyz="-0.052159 -0.044445 0.049943" rpy="0 0 0"/>
+      <origin xyz="-0.043476 -0.044445 0.049183" rpy="0 0 0"/>
       <geometry>
         <mesh filename="package://mini_pupper_description/meshes/lf3.stl" scale="1 1 1"/>
@@ -86,8 +86,8 @@
   </link>
   <link name="rf1">
-      <inertial>
+    <inertial>
       <origin xyz="0.020106742599110078 -0.00233237781568562 0.006497900858401761" rpy="0 0 0"/>
       <mass value="0.020769549324466178"/>
-      <inertia ixx="2e-06" iyy="4e-06" izz="3e-06" ixy="0.0" iyz="-0.0" ixz="-0.0"/>
+      <inertia ixx="2e-06" iyy="4e-06" izz="3e-06" ixy="0.0" iyz="0.0" ixz="0.0"/>
     </inertial>
     <visual>
@@ -107,7 +107,7 @@
   <link name="rf2">
     <inertial>
-      <origin xyz="-4.1025190424676117e-07 -0.0009866275794596438 -0.018261345629717353" rpy="0 0 0"/>
+      <origin xyz="-0.00317137334512671 -0.000986627579459616 -0.01798392230653304" rpy="0 0 0"/>
       <mass value="0.0019057729924780605"/>
-      <inertia ixx="0.0" iyy="0.0" izz="0.0" ixy="-0.0" iyz="-0.0" ixz="-0.0"/>
+      <inertia ixx="0.0" iyy="0.0" izz="0.0" ixy="0.0" iyz="0.0" ixz="0.0"/>
     </inertial>
     <visual>
@@ -127,10 +127,10 @@
   <link name="rf3">
     <inertial>
-      <origin xyz="0.0007030898236521158 -0.003457422744677939 -0.016230262912113935" rpy="0 0 0"/>
+      <origin xyz="0.006211719758792998 -0.0034574884973188197 -0.01500899883342268" rpy="0 0 0"/>
       <mass value="0.001143490701517533"/>
-      <inertia ixx="1e-06" iyy="1e-06" izz="0.0" ixy="0.0" iyz="-0.0" ixz="0.0"/>
-    </inertial>
-    <visual>
-      <origin xyz="-0.052165 0.043955 0.049943" rpy="0 0 0"/>
+      <inertia ixx="1e-06" iyy="1e-06" izz="0.0" ixy="0.0" iyz="0.0" ixz="0.0"/>
+    </inertial>
+    <visual>
+      <origin xyz="-0.043482 0.043955 0.049184" rpy="0 0 0"/>
       <geometry>
         <mesh filename="package://mini_pupper_description/meshes/rf3.stl" scale="1 1 1"/>
@@ -139,5 +139,5 @@
     </visual>
     <collision>
-      <origin xyz="-0.052165 0.043955 0.049943" rpy="0 0 0"/>
+      <origin xyz="-0.043482 0.043955 0.049184" rpy="0 0 0"/>
       <geometry>
         <mesh filename="package://mini_pupper_description/meshes/rf3.stl" scale="1 1 1"/>
@@ -149,5 +149,5 @@
       <origin xyz="-0.020107177922528044 -0.0023288309787250286 0.006502376356642127" rpy="0 0 0"/>
       <mass value="0.020769549324363486"/>
-      <inertia ixx="2e-06" iyy="4e-06" izz="3e-06" ixy="-0.0" iyz="-0.0" ixz="-0.0"/>
+      <inertia ixx="2e-06" iyy="4e-06" izz="3e-06" ixy="0.0" iyz="0.0" ixz="0.0"/>
     </inertial>
     <visual>
@@ -167,7 +167,7 @@
   <link name="rb2">
     <inertial>
-      <origin xyz="-2.5070667000748337e-08 -0.000996585764066693 -0.018260149861185754" rpy="0 0 0"/>
+      <origin xyz="-0.0031709881638501275 -0.0009964344348111775 -0.017982726579309202" rpy="0 0 0"/>
       <mass value="0.0019057729926311429"/>
-      <inertia ixx="0.0" iyy="0.0" izz="0.0" ixy="-0.0" iyz="-0.0" ixz="-0.0"/>
+      <inertia ixx="0.0" iyy="0.0" izz="0.0" ixy="0.0" iyz="0.0" ixz="0.0"/>
     </inertial>
     <visual>
@@ -187,10 +187,10 @@
   <link name="rb3">
     <inertial>
-      <origin xyz="0.0007031309185970697 -0.0034624258831375196 -0.016220094399306113" rpy="0 0 0"/>
+      <origin xyz="0.006208573190273861 -0.0034623583329196975 -0.015001217060300935" rpy="0 0 0"/>
       <mass value="0.0011440535724654094"/>
-      <inertia ixx="1e-06" iyy="1e-06" izz="0.0" ixy="0.0" iyz="-0.0" ixz="0.0"/>
-    </inertial>
-    <visual>
-      <origin xyz="0.068367 0.043983 0.049932" rpy="0 0 0"/>
+      <inertia ixx="1e-06" iyy="1e-06" izz="0.0" ixy="0.0" iyz="0.0" ixz="0.0"/>
+    </inertial>
+    <visual>
+      <origin xyz="0.077049 0.043982 0.049173" rpy="0 0 0"/>
       <geometry>
         <mesh filename="package://mini_pupper_description/meshes/rb3.stl" scale="1 1 1"/>
@@ -199,5 +199,5 @@
     </visual>
     <collision>
-      <origin xyz="0.068367 0.043983 0.049932" rpy="0 0 0"/>
+      <origin xyz="0.077049 0.043982 0.049173" rpy="0 0 0"/>
       <geometry>
         <mesh filename="package://mini_pupper_description/meshes/rb3.stl" scale="1 1 1"/>
@@ -209,5 +209,5 @@
       <origin xyz="-0.020109716415830967 0.0023317718989125207 0.006499556305653081" rpy="0 0 0"/>
       <mass value="0.020769030189864354"/>
-      <inertia ixx="2e-06" iyy="4e-06" izz="3e-06" ixy="0.0" iyz="0.0" ixz="-0.0"/>
+      <inertia ixx="2e-06" iyy="4e-06" izz="3e-06" ixy="0.0" iyz="0.0" ixz="0.0"/>
     </inertial>
     <visual>
@@ -227,7 +227,7 @@
   <link name="lb2">
     <inertial>
-      <origin xyz="-2.486178994620669e-08 0.0009860564153100007 -0.01826134562993383" rpy="0 0 0"/>
+      <origin xyz="-0.0031709879518865836 0.0009860564153100285 -0.01798392227051571" rpy="0 0 0"/>
       <mass value="0.0019057729925095609"/>
-      <inertia ixx="0.0" iyy="0.0" izz="0.0" ixy="0.0" iyz="0.0" ixz="-0.0"/>
+      <inertia ixx="0.0" iyy="0.0" izz="0.0" ixy="0.0" iyz="0.0" ixz="0.0"/>
     </inertial>
     <visual>
@@ -247,10 +247,10 @@
   <link name="lb3">
     <inertial>
-      <origin xyz="0.0007030123702261443 0.0034519487133846394 -0.016218113385159758" rpy="0 0 0"/>
+      <origin xyz="0.006208905683926957 0.0034523757482988054 -0.015005654191541921" rpy="0 0 0"/>
       <mass value="0.001144346207072784"/>
-      <inertia ixx="1e-06" iyy="1e-06" izz="0.0" ixy="-0.0" iyz="0.0" ixz="0.0"/>
-    </inertial>
-    <visual>
-      <origin xyz="0.068367 -0.044445 0.049943" rpy="0 0 0"/>
+      <inertia ixx="1e-06" iyy="1e-06" izz="0.0" ixy="0.0" iyz="0.0" ixz="0.0"/>
+    </inertial>
+    <visual>
+      <origin xyz="0.077049 -0.044445 0.049184" rpy="0 0 0"/>
       <geometry>
         <mesh filename="package://mini_pupper_description/meshes/lb3.stl" scale="1 1 1"/>
@@ -259,5 +259,5 @@
     </visual>
     <collision>
-      <origin xyz="0.068367 -0.044445 0.049943" rpy="0 0 0"/>
+      <origin xyz="0.077049 -0.044445 0.049184" rpy="0 0 0"/>
       <geometry>
         <mesh filename="package://mini_pupper_description/meshes/lb3.stl" scale="1 1 1"/>
@@ -269,5 +269,5 @@
       <origin xyz="-0.005538678480206852 -0.00020424196520824284 0.020222593513387798" rpy="0 0 0"/>
       <mass value="0.00785515871148119"/>
-      <inertia ixx="5e-06" iyy="2e-06" izz="4e-06" ixy="-0.0" iyz="-0.0" ixz="-0.0"/>
+      <inertia ixx="5e-06" iyy="2e-06" izz="4e-06" ixy="0.0" iyz="0.0" ixz="0.0"/>
     </inertial>
     <visual>
@@ -329,5 +329,5 @@
       <origin xyz="0.008233541174180986 -0.002138369786547657 -0.00030110978110910874" rpy="0 0 0"/>
       <mass value="0.0019746031301169403"/>
-      <inertia ixx="0.0" iyy="3e-06" izz="4e-06" ixy="-0.0" iyz="0.0" ixz="0.0"/>
+      <inertia ixx="0.0" iyy="3e-06" izz="4e-06" ixy="0.0" iyz="0.0" ixz="0.0"/>
     </inertial>
     <visual>
@@ -347,10 +347,10 @@
   <link name="rffoot">
     <inertial>
-      <origin xyz="-0.0024634044240561814 -2.8557999392359035e-07 0.007801816226636768" rpy="0 0 0"/>
+      <origin xyz="-0.004983173489839052 -2.855799938611403e-07 0.006488367917121082" rpy="0 0 0"/>
       <mass value="0.0014053107976262874"/>
-      <inertia ixx="0.0" iyy="0.0" izz="0.0" ixy="0.0" iyz="-0.0" ixz="-0.0"/>
-    </inertial>
-    <visual>
-      <origin xyz="-0.056689 0.047705 0.109514" rpy="0 0 0"/>
+      <inertia ixx="0.0" iyy="0.0" izz="0.0" ixy="0.0" iyz="0.0" ixz="0.0"/>
+    </inertial>
+    <visual>
+      <origin xyz="-0.068108 0.047705 0.103614" rpy="0 0 0"/>
       <geometry>
         <mesh filename="package://mini_pupper_description/meshes/rffoot.stl" scale="1 1 1"/>
@@ -359,5 +359,5 @@
     </visual>
     <collision>
-      <origin xyz="-0.056689 0.047705 0.109514" rpy="0 0 0"/>
+      <origin xyz="-0.068108 0.047705 0.103614" rpy="0 0 0"/>
       <geometry>
         <mesh filename="package://mini_pupper_description/meshes/rffoot.stl" scale="1 1 1"/>
@@ -367,10 +367,10 @@
   <link name="rbfoot">
     <inertial>
-      <origin xyz="-0.0024630192318816357 4.2051173794327434e-06 0.0078011683948505245" rpy="0 0 0"/>
+      <origin xyz="-0.004982788301465979 3.706995898918042e-06 0.006488719406103974" rpy="0 0 0"/>
       <mass value="0.0014053107976262874"/>
-      <inertia ixx="0.0" iyy="0.0" izz="0.0" ixy="-0.0" iyz="-0.0" ixz="-0.0"/>
-    </inertial>
-    <visual>
-      <origin xyz="0.063843 0.047765 0.1095" rpy="0 0 0"/>
+      <inertia ixx="0.0" iyy="0.0" izz="0.0" ixy="0.0" iyz="0.0" ixz="0.0"/>
+    </inertial>
+    <visual>
+      <origin xyz="0.052424 0.047762 0.103601" rpy="0 0 0"/>
       <geometry>
         <mesh filename="package://mini_pupper_description/meshes/rbfoot.stl" scale="1 1 1"/>
@@ -379,5 +379,5 @@
     </visual>
     <collision>
-      <origin xyz="0.063843 0.047765 0.1095" rpy="0 0 0"/>
+      <origin xyz="0.052424 0.047762 0.103601" rpy="0 0 0"/>
       <geometry>
         <mesh filename="package://mini_pupper_description/meshes/rbfoot.stl" scale="1 1 1"/>
@@ -387,10 +387,10 @@
   <link name="lbfoot">
     <inertial>
-      <origin xyz="-0.0024630193952935586 -2.855826621572799e-07 0.00780181622349041" rpy="0 0 0"/>
+      <origin xyz="-0.004982788451759437 -2.855826620323798e-07 0.0064883680140642025" rpy="0 0 0"/>
       <mass value="0.0014053107976262874"/>
-      <inertia ixx="0.0" iyy="0.0" izz="0.0" ixy="0.0" iyz="-0.0" ixz="-0.0"/>
-    </inertial>
-    <visual>
-      <origin xyz="0.063843 -0.048195 0.109514" rpy="0 0 0"/>
+      <inertia ixx="0.0" iyy="0.0" izz="0.0" ixy="0.0" iyz="0.0" ixz="0.0"/>
+    </inertial>
+    <visual>
+      <origin xyz="0.052424 -0.048195 0.103614" rpy="0 0 0"/>
       <geometry>
         <mesh filename="package://mini_pupper_description/meshes/lbfoot.stl" scale="1 1 1"/>
@@ -399,5 +399,5 @@
     </visual>
     <collision>
-      <origin xyz="0.063843 -0.048195 0.109514" rpy="0 0 0"/>
+      <origin xyz="0.052424 -0.048195 0.103614" rpy="0 0 0"/>
       <geometry>
         <mesh filename="package://mini_pupper_description/meshes/lbfoot.stl" scale="1 1 1"/>
@@ -407,10 +407,10 @@
   <link name="lffoot">
     <inertial>
-      <origin xyz="-0.002463300234335934 -2.8611328430766525e-07 0.00780127458383767" rpy="0 0 0"/>
+      <origin xyz="-0.004983499344395154 -2.861132842799097e-07 0.006488888240325896" rpy="0 0 0"/>
       <mass value="0.0014053107976262874"/>
-      <inertia ixx="0.0" iyy="0.0" izz="0.0" ixy="0.0" iyz="-0.0" ixz="-0.0"/>
-    </inertial>
-    <visual>
-      <origin xyz="-0.056689 -0.048195 0.109513" rpy="0 0 0"/>
+      <inertia ixx="0.0" iyy="0.0" izz="0.0" ixy="0.0" iyz="0.0" ixz="0.0"/>
+    </inertial>
+    <visual>
+      <origin xyz="-0.068108 -0.048195 0.103611" rpy="0 0 0"/>
       <geometry>
         <mesh filename="package://mini_pupper_description/meshes/lffoot.stl" scale="1 1 1"/>
@@ -419,5 +419,5 @@
     </visual>
     <collision>
-      <origin xyz="-0.056689 -0.048195 0.109513" rpy="0 0 0"/>
+      <origin xyz="-0.068108 -0.048195 0.103611" rpy="0 0 0"/>
       <geometry>
         <mesh filename="package://mini_pupper_description/meshes/lffoot.stl" scale="1 1 1"/>
@@ -469,5 +469,5 @@
       <origin xyz="0.002219644336096324 -0.008605630927951344 -0.002709000699399786" rpy="0 0 0"/>
       <mass value="0.002396251664132183"/>
-      <inertia ixx="0.0" iyy="0.0" izz="0.0" ixy="-0.0" iyz="-0.0" ixz="0.0"/>
+      <inertia ixx="0.0" iyy="0.0" izz="0.0" ixy="0.0" iyz="0.0" ixz="0.0"/>
     </inertial>
     <visual>
@@ -489,5 +489,5 @@
       <origin xyz="0.0022200295152449145 -0.008607013686777375 -0.0027033986949916797" rpy="0 0 0"/>
       <mass value="0.002396251664132183"/>
-      <inertia ixx="0.0" iyy="0.0" izz="0.0" ixy="-0.0" iyz="-0.0" ixz="0.0"/>
+      <inertia ixx="0.0" iyy="0.0" izz="0.0" ixy="0.0" iyz="0.0" ixz="0.0"/>
     </inertial>
     <visual>
@@ -507,10 +507,10 @@
   <link name="Shell_Leg_Upper_LeftSide_1">
     <inertial>
-      <origin xyz="-0.0026521199361419917 0.00790352811362325 0.004979527414372081" rpy="0 0 0"/>
-      <mass value="0.00223142111318912"/>
-      <inertia ixx="1e-06" iyy="1e-06" izz="0.0" ixy="0.0" iyz="-0.0" ixz="0.0"/>
-    </inertial>
-    <visual>
-      <origin xyz="-0.052162 -0.044445 0.018943" rpy="0 0 0"/>
+      <origin xyz="-0.001747332142694763 0.00790352811362327 0.005364507913861985" rpy="0 0 0"/>
+      <mass value="0.0022314211131891203"/>
+      <inertia ixx="1e-06" iyy="1e-06" izz="0.0" ixy="0.0" iyz="-0.0" ixz="-0.0"/>
+    </inertial>
+    <visual>
+      <origin xyz="-0.048863 -0.044445 0.018654" rpy="0 0 0"/>
       <geometry>
         <mesh filename="package://mini_pupper_description/meshes/Shell_Leg_Upper_LeftSide_1.stl" scale="1 1 1"/>
@@ -519,5 +519,5 @@
     </visual>
     <collision>
-      <origin xyz="-0.052162 -0.044445 0.018943" rpy="0 0 0"/>
+      <origin xyz="-0.048863 -0.044445 0.018654" rpy="0 0 0"/>
       <geometry>
         <mesh filename="package://mini_pupper_description/meshes/Shell_Leg_Upper_LeftSide_1.stl" scale="1 1 1"/>
@@ -527,10 +527,10 @@
   <link name="Shell_Leg_Upper_LeftSide_2">
     <inertial>
-      <origin xyz="-0.002652484362897875 0.007903528639619295 0.004979527279084269" rpy="0 0 0"/>
-      <mass value="0.00223142111318912"/>
-      <inertia ixx="1e-06" iyy="1e-06" izz="0.0" ixy="0.0" iyz="-0.0" ixz="0.0"/>
-    </inertial>
-    <visual>
-      <origin xyz="0.068367 -0.044445 0.018943" rpy="0 0 0"/>
+      <origin xyz="-0.001747730780760487 0.007903528639619323 0.005365117008527457" rpy="0 0 0"/>
+      <mass value="0.0022314211131891203"/>
+      <inertia ixx="1e-06" iyy="1e-06" izz="0.0" ixy="0.0" iyz="-0.0" ixz="-0.0"/>
+    </inertial>
+    <visual>
+      <origin xyz="0.071666 -0.044445 0.018655" rpy="0 0 0"/>
       <geometry>
         <mesh filename="package://mini_pupper_description/meshes/Shell_Leg_Upper_LeftSide_2.stl" scale="1 1 1"/>
@@ -539,5 +539,5 @@
     </visual>
     <collision>
-      <origin xyz="0.068367 -0.044445 0.018943" rpy="0 0 0"/>
+      <origin xyz="0.071666 -0.044445 0.018655" rpy="0 0 0"/>
       <geometry>
         <mesh filename="package://mini_pupper_description/meshes/Shell_Leg_Upper_LeftSide_2.stl" scale="1 1 1"/>
@@ -547,10 +547,10 @@
   <link name="Shell_Leg_Upper_RightSide_1">
     <inertial>
-      <origin xyz="-0.0027172440375204526 -0.007907075713007534 0.004991745926148535" rpy="0 0 0"/>
-      <mass value="0.0022016115622538724"/>
-      <inertia ixx="1e-06" iyy="1e-06" izz="0.0" ixy="-0.0" iyz="0.0" ixz="0.0"/>
-    </inertial>
-    <visual>
-      <origin xyz="-0.052165 0.043955 0.018943" rpy="0 0 0"/>
+      <origin xyz="-0.0018083907227202795 -0.007907075713007514 0.005388328467850496" rpy="0 0 0"/>
+      <mass value="0.002201611562253873"/>
+      <inertia ixx="1e-06" iyy="1e-06" izz="0.0" ixy="-0.0" iyz="0.0" ixz="-0.0"/>
+    </inertial>
+    <visual>
+      <origin xyz="-0.048865 0.043955 0.018655" rpy="0 0 0"/>
       <geometry>
         <mesh filename="package://mini_pupper_description/meshes/Shell_Leg_Upper_RightSide_1.stl" scale="1 1 1"/>
@@ -559,5 +559,5 @@
     </visual>
     <collision>
-      <origin xyz="-0.052165 0.043955 0.018943" rpy="0 0 0"/>
+      <origin xyz="-0.048865 0.043955 0.018655" rpy="0 0 0"/>
       <geometry>
         <mesh filename="package://mini_pupper_description/meshes/Shell_Leg_Upper_RightSide_1.stl" scale="1 1 1"/>
@@ -567,10 +567,10 @@
   <link name="Shell_Leg_Upper_RightSide_2">
     <inertial>
-      <origin xyz="-0.002716858856166446 -0.007903712439730225 0.004996352480544097" rpy="0 0 0"/>
-      <mass value="0.0022016115622538724"/>
-      <inertia ixx="1e-06" iyy="1e-06" izz="0.0" ixy="-0.0" iyz="0.0" ixz="0.0"/>
-    </inertial>
-    <visual>
-      <origin xyz="0.068367 0.043966 0.018932" rpy="0 0 0"/>
+      <origin xyz="-0.0018090055415128231 -0.007904339012704771 0.005392934920359041" rpy="0 0 0"/>
+      <mass value="0.002201611562253873"/>
+      <inertia ixx="1e-06" iyy="1e-06" izz="0.0" ixy="-0.0" iyz="0.0" ixz="-0.0"/>
+    </inertial>
+    <visual>
+      <origin xyz="0.071666 0.043965 0.018644" rpy="0 0 0"/>
       <geometry>
         <mesh filename="package://mini_pupper_description/meshes/Shell_Leg_Upper_RightSide_2.stl" scale="1 1 1"/>
@@ -579,5 +579,5 @@
     </visual>
     <collision>
-      <origin xyz="0.068367 0.043966 0.018932" rpy="0 0 0"/>
+      <origin xyz="0.071666 0.043965 0.018644" rpy="0 0 0"/>
       <geometry>
         <mesh filename="package://mini_pupper_description/meshes/Shell_Leg_Upper_RightSide_2.stl" scale="1 1 1"/>
@@ -621,12 +621,12 @@
     <parent link="lf1"/>
     <child link="lf2"/>
-    <axis xyz="0.0 1.0 -0.0"/>
+    <axis xyz="0.0 1.0 0.0"/>
     <limit upper="3.141593" lower="-3.141593" effort="5" velocity="1.5"/>
   </joint>
   <joint name="lf2_lf3" type="revolute">
-    <origin xyz="-6e-06 0.003 -0.05" rpy="0 0 0"/>
+    <origin xyz="-0.008689 0.003 -0.04924" rpy="0 0 0"/>
     <parent link="lf2"/>
     <child link="lf3"/>
-    <axis xyz="0.0 1.0 -0.0"/>
+    <axis xyz="0.0 1.0 0.0"/>
     <limit upper="3.141593" lower="-3.141593" effort="5" velocity="1.5"/>
   </joint>
@@ -646,5 +646,5 @@
   </joint>
   <joint name="rf2_rf3" type="revolute">
-    <origin xyz="0.0 -0.003 -0.05" rpy="0 0 0"/>
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